File: Util/stomp-chargepump/stomp-chargepump.kicad_pcb (KiCad board)
At the start: 2 copper layers, 52.7 x 28.6 mm, 15 parts, among them J1 to-effect, J2 to-effect, J3 from-top-jacks, J4 to-effect, U1 MAX1044

Commit message: missing files
Parts:
- removed J2, J4: to-effect, Connector_PinHeader_2.54mm:PinHeader_1x04_P2.54mm_Vertical
- J1: footprint Connector_PinHeader_2.54mm:PinHeader_1x04_P2.54mm_Vertical -> Connector_PinHeader_2.54mm:PinHeader_1x06_P2.54mm_Vertical
- moved D2 0.30 mm to (123.7, 75.7)
- moved J1 0.21 mm to (114.8, 70.5)
Connections:
- J1 pad 1: -9V -> 18V
- J1 pad 2: SEND -> -9V
- J1 pad 3: RECV -> +9V
- J1 pad 4: GND -> SEND
Routing:
- net RECV: track 39.7 -> 14.6 mm
- net SEND: track 52.4 -> 27.7 mm
- net 18V: track 74.6 -> 86.6 mm
- net IN: track 29.4 -> 35.4 mm
- net -9V: track 30.2 -> 34.1 mm
- net +9V: track 37.6 -> 39.9 mm
- net OUT: track 23.7 -> 22.8 mm, vias 1 -> 0
