File: Overdrive/ecstacy/ecstacy.kicad_pcb (KiCad board)
At the start: 2 copper layers, 59.3 x 36.8 mm, 41 parts, among them J1 Conn_01x04_Pin, SW1 SW_DPDT_x2, U1 NJM4558

Commit message: fix to badmonkey -- pedal works but the schematic this was based on does not seem right.   There's a voltage offset on the input when engaged, and this messes with it in the pedal chain.
Changed lines of the file:
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@@
         (effects (font (size 1 1) (thickness 0.15)))
     )
-    (fp_text value "22n" (at 2.5 2.5) (layer "F.Fab")
+    (fp_text value "22n" (at 2.5 0.55) (layer "F.SilkS")
         (effects (font (size 1 1) (thickness 0.15)))
     )
