File: Distortion/bigmuff/bmp-ramshead.kicad_pcb (KiCad board)
At the start: 2 copper layers, 58 x 43.6 mm, 46 parts, among them J1 Conn_01x04_Female, Q1 2N5089, Q2 2N5089, Q3 2N5089, Q4 2N5089

Commit message: added ejfuzzface
Changed lines of the file:
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@@
-    (effects (font (size 1.5 1.5) (thickness 0.3) bold) (justify left bottom))
-  )
-  (gr_text "NOT VERIFIED, though schematic is verified." (at 53.88 49.14) (layer "F.SilkS")
     (effects (font (size 1.5 1.5) (thickness 0.3) bold) (justify left bottom))
   )
@@
     (effects (font (size 1 1) (thickness 0.15)))
   )
+  (gr_text "NOT VERIFIED, though schematic is verified." (at 53.36 46.01) (layer "F.Fab")
+    (effects (font (size 1.5 1.5) (thickness 0.3) bold) (justify left bottom))
+  )
   (segment (start 97.4574 82.8874) (end 96.35 81.78) (width 0.25) (layer "B.Cu") (net 1))
