File: Distortion/bigmuff/bmp-ramshead.kicad_pcb (KiCad board)
At the start: 2 copper layers, 58 x 43.6 mm, 46 parts, among them J1 Conn_01x04_Female, Q1 2N5089, Q2 2N5089, Q3 2N5089, Q4 2N5089

Commit message: Changed the silkscreen layer
Parts:
- D1, D2, D3, D4: value 1n4148 -> 4148
Other:
- board text added: "BMP ramshead"
Changed lines of the file:
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@@
         (effects (font (size 0.7 0.7) (thickness 0.1)))
     )
-    (fp_text value "1n4148" (at 4.24 0.75) (layer "F.SilkS")
+    (fp_text value "4148" (at 4.24 0.75) (layer "F.SilkS")
         (effects (font (size 0.7 0.7) (thickness 0.1)))
     )
@@
     (property "ki_keywords" "R res resistor")
     (attr through_hole)
-    (fp_text reference "R17" (at 5.08 -2.37) (layer "F.SilkS")
-        (effects (font (size 0.7 0.7) (thickness 0.1)))
-    )
-    (fp_text value "33k" (at 5.08 2.37) (layer "F.SilkS")
+    (fp_text reference "R17" (at 3.15 -0.79) (layer "F.SilkS")
+        (effects (font (size 0.7 0.7) (thickness 0.1)))
+    )
+    (fp_text value "33k" (at 5.74 0.68) (layer "F.SilkS")
         (effects (font (size 0.7 0.7) (thickness 0.1)))
     )
@@
     (property "ki_keywords" "connector")
     (attr through_hole)
-    (fp_text reference "J1" (at 0 -2.33 90) (layer "F.SilkS")
+    (fp_text reference "J1" (at 0 -2.33 90) (layer "F.SilkS") hide
         (effects (font (size 0.7 0.7) (thickness 0.1)))
     )
@@
     (property "ki_keywords" "R res resistor")
     (attr through_hole)
-    (fp_text reference "R18" (at 5.08 -2.37) (layer "F.SilkS")
+    (fp_text reference "R18" (at 3.07 -0.61) (layer "F.SilkS")
         (effects (font (size 0.7 0.7) (thickness 0.1)))
     )
@@
     (property "ki_keywords" "diode")
     (attr through_hole)
-    (fp_text reference "D3" (at 4.82 -0.37) (layer "F.SilkS")
-        (effects (font (size 0.7 0.7) (thickness 0.1)))
-    )
-    (fp_text value "1n4148" (at 4.74 0.55) (layer "F.SilkS")
+    (fp_text reference "D3" (at 3.45 -0.79) (layer "F.SilkS")
+        (effects (font (size 0.7 0.7) (thickness 0.1)))
+    )
+    (fp_text value "4148" (at 4.74 0.55) (layer "F.SilkS")
         (effects (font (size 0.7 0.7) (thickness 0.1)))
     )
@@
         (effects (font (size 1 1) (thickness 0.15)))
     )
-    (fp_text user "K" (at 0 -1.9) (layer "F.Fab")
+    (fp_text user "K" (at 0 -1.9) (layer "F.Fab") hide
         (effects (font (size 1 1) (thickness 0.15)))
     )
@@
     (property "ki_keywords" "NPN Transistor")
     (attr through_hole)
-    (fp_text reference "Q3" (at 1.27 -3.56) (layer "F.SilkS")
-        (effects (font (size 1 1) (thickness 0.15)))
-    )
-    (fp_text value "2N5089" (at 1.27 2.79) (layer "F.Fab")
-        (effects (font (size 1 1) (thickness 0.15)))
+    (fp_text reference "Q3" (at 1.17 -1.54) (layer "F.SilkS")
+        (effects (font (size 0.8 0.8) (thickness 0.15)))
+    )
+    (fp_text value "2N5089" (at 1.23 2.55) (layer "F.SilkS")
+        (effects (font (size 0.7 0.7) (thickness 0.15)))
     )
     (fp_text user "${REFERENCE}" (at 1.27 0) (layer "F.Fab")
@@
     (property "ki_keywords" "diode")
     (attr through_hole)
-    (fp_text reference "D2" (at 3.81 -1.47) (layer "F.SilkS")
-        (effects (font (size 0.7 0.7) (thickness 0.1)))
-    )
-    (fp_text value "1n4148" (at 4.08 0.62) (layer "F.SilkS")
+    (fp_text reference "D2" (at 4.04 -0.68) (layer "F.SilkS")
+        (effects (font (size 0.7 0.7) (thickness 0.1)))
+    )
+    (fp_text value "4148" (at 4.08 0.62) (layer "F.SilkS")
         (effects (font (size 0.7 0.7) (thickness 0.1)))
     )
@@
         (effects (font (size 0.7 0.7) (thickness 0.1)))
     )
-    (fp_text value "2N5089" (at 0.84 1.22) (layer "F.SilkS")
+    (fp_text value "2N5089" (at 1.06 2.45) (layer "F.SilkS")
         (effects (font (size 0.7 0.7) (thickness 0.1)))
     )
@@
         (effects (font (size 0.7 0.7) (thickness 0.1)))
     )
-    (fp_text value "2N5089" (at 1.05 1.22) (layer "F.SilkS")
+    (fp_text value "2N5089" (at 1.12 2.44) (layer "F.SilkS")
         (effects (font (size 0.7 0.7) (thickness 0.1)))
     )
@@
     (property "ki_keywords" "R res resistor")
     (attr through_hole)
-    (fp_text reference "R16" (at 5.08 -2.37) (layer "F.SilkS")
-        (effects (font (size 0.7 0.7) (thickness 0.1)))
-    )
-    (fp_text value "33k" (at 5.08 2.37) (layer "F.SilkS")
+    (fp_text reference "R16" (at 3.39 -0.43) (layer "F.SilkS")
+        (effects (font (size 0.7 0.7) (thickness 0.1)))
+    )
+    (fp_text value "33k" (at 6.33 0.63) (layer "F.SilkS")
         (effects (font (size 0.7 0.7) (thickness 0.1)))
     )
@@
     (property "ki_keywords" "R res resistor")
     (attr through_hole)
-    (fp_text reference "R5" (at 3.39 -0.93) (layer "F.SilkS")
+    (fp_text reference "R5" (at 3.38 -0.61) (layer "F.SilkS")
         (effects (font (size 0.7 0.7) (thickness 0.1)))
     )
@@
         (effects (font (size 0.7 0.7) (thickness 0.1)))
     )
-    (fp_text value "2N5089" (at 1.24 1.29) (layer "F.SilkS")
+    (fp_text value "2N5089" (at 1.25 2.42) (layer "F.SilkS")
         (effects (font (size 0.7 0.7) (thickness 0.1)))
     )
@@
         (effects (font (size 0.7 0.7) (thickness 0.1)))
     )
-    (fp_text value "1n4148" (at 4.37 0.71) (layer "F.SilkS")
+    (fp_text value "4148" (at 4.37 0.71) (layer "F.SilkS")
         (effects (font (size 0.7 0.7) (thickness 0.1)))
     )
@@
         (effects (font (size 1 1) (thickness 0.15)) (justify mirror))
     )
-    (fp_text value "A100k" (at 3.54 -7.69 -270) (layer "B.Fab")
+    (fp_text value "A100k" (at 3.54 -7.69 90) (layer "B.SilkS")
         (effects (font (size 1 1) (thickness 0.15)) (justify mirror))
     )
@@
         (effects (font (size 1 1) (thickness 0.15)) (justify mirror))
     )
-    (fp_text value "A100k" (at 3.625 -7.31 -270) (layer "B.Fab")
+    (fp_text value "A100k" (at 3.625 -7.31 90) (layer "B.SilkS")
         (effects (font (size 1 1) (thickness 0.15)) (justify mirror))
     )
@@
         (effects (font (size 1 1) (thickness 0.15)) (justify mirror))
     )
-    (fp_text value "A100k" (at 3.39 -7.58 -270) (layer "B.Fab")
+    (fp_text value "A100k" (at 3.39 -7.58 90) (layer "B.SilkS")
         (effects (font (size 1 1) (thickness 0.15)) (justify mirror))
     )
@@
   (gr_line (start 88.6 50) (end 88.6 90)
     (stroke (width 0.1) (type solid)) (layer "F.Fab"))
-  (gr_line (start 79 50) (end 79 90)
-    (stroke (width 0.1) (type solid)) (layer "User.1"))
-  (gr_line (start 99 50) (end 99 90)
-    (stroke (width 0.1) (type solid)) (layer "User.1"))
-  (gr_line (start 59 50) (end 59 90)
-    (stroke (width 0.1) (type solid)) (layer "User.1"))
   (gr_text "vol" (at 57.29 54.3) (layer "F.SilkS")
     (effects (font (size 1.5 1.5) (thickness 0.3) bold) (justify left bottom))
@@
     (effects (font (size 1.5 1.5) (thickness 0.3) bold) (justify left bottom))
   )
+  (gr_text "BMP\nramshead" (at 95.78 64.59) (layer "F.SilkS")
+    (effects (font (size 1 1) (thickness 0.15)) (justify left bottom))
+  )
   (gr_text "125b-58x40" (at 56 48) (layer "F.Fab")
